Commit message: Wall height increased

File: week 1/table(1).urdf (robot description, URDF)
Before this commit: robot table, 10 links, 9 joints
Links:
- link Xneg_Yneg: geometry collision box size=0.3 0.05 0.3; visual box size=0.3 0.05 0.4
- link Xneg_Ypos: geometry collision box size=0.3 0.05 0.3; visual box size=0.3 0.05 0.4
- link Xpos_Yneg: geometry collision box size=0.3 0.05 0.3; visual box size=0.3 0.05 0.4
- link Xpos_Ypos: geometry collision box size=0.3 0.05 0.3; visual box size=0.3 0.05 0.4
- link Y_N: geometry collision box size=1.8 0.05 0.3; visual box size=1.8 0.05 0.4
- link Y_P: geometry collision box size=1.8 0.05 0.3; visual box size=1.8 0.05 0.4

Commit message: fixed inertial properties

File: week 1/table(1).urdf (robot description, URDF)
Before this commit: robot table, 10 links, 9 joints
Links:
- removed link baseE
- removed link baseF
- removed link baseG
- link Xneg_Yneg: mass None -> 25
- link Xneg_Ypos: mass None -> 25
- link Xpos_Yneg: mass None -> 25
- link Xpos_Ypos: mass None -> 25
- link Y_N: mass None -> 50
- link Y_P: mass None -> 50
- link base: mass None -> 50; geometry collision box size=1.8 1 0.30; visual box size=1.8 1 0.30
Joints:
- removed joint base_to_base1
- removed joint base_to_base2
- removed joint base_to_base3
