Commit message: new hitbot at place of kuka

File: week 1/hitbot.urdf (robot description, URDF)
Before this commit: robot hitter, 2 links, 1 joints
Links:
- removed link base_link
- removed link right_leg
- added link base, mass 100; collision box size=0.9 0.05 0.008; visual box size=0.9 0.05 0.008
- added link base_R, mass 100; collision box size=0.9 0.05 0.008; visual box size=0.9 0.05 0.008
- added link extension, mass 1; collision cylinder length=0.08 radius=0.015; visual cylinder length=0.08 radius=0.015
- added link hockey, mass 1; collision cylinder length=0.04 radius=0.06; visual cylinder length=0.04 radius=0.06
- added link slider, mass 5; collision box size=0.08 1.05 0.02; visual box size=0.08 1.05 0.02
Joints:
- removed joint base_to_right_leg
- added joint base_L_to_base_R: type fixed, parent base, child base_R, origin xyz=0 0 0
- added joint base_to_slider: type prismatic, parent base, child slider, origin xyz=0 0 0, axis 1 0 0, limit lower=-0.38 upper=0.38 effort=100.0 velocity=0.9
- added joint extension_to_hockey: type fixed, parent extension, child hockey, origin xyz=0 0 0
- added joint slider_to_extension: type prismatic, parent slider, child extension, origin xyz=0 0 -0.02, axis 0 1 0, limit lower=-0.44 upper=0.44 effort=100.0 velocity=0.9

Commit message: Add files via upload

File: week 1/hitbot.urdf (robot description, URDF)
Before this commit: robot slider_bot, 5 links, 4 joints
Links:
- link hockey: geometry collision cylinder length=0.04 radius=0.08; visual cylinder length=0.04 radius=0.08

Commit message: Add files via upload

File: week 1/hitbot.urdf (robot description, URDF)
Before this commit: robot slider_bot, 5 links, 4 joints
Links:
- link hockey: mass 1 -> 0.2

File: week 1/puck(1).urdf (robot description, URDF)
Before this commit: robot puck, 1 links, 0 joints
Links:
- link base: geometry collision cylinder length=0.02 radius=0.06; visual cylinder length=0.02 radius=0.06
